File: 42Keys/chocorne/chococorne.kicad_pcb (KiCad board)
At the start: 2 copper layers, 130 x 87.7 mm, 63 parts, among them J1 MJ-4PP-9, J2 OLED, SW1 SW_PUSH, SW10 SW_PUSH, SW11 SW_PUSH, SW12 SW_PUSH, SW13 SW_PUSH, SW14 SW_PUSH, SW15 SW_PUSH, SW16 SW_PUSH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

Commit message: Add legend
Other:
- board text added: "ChocoCorne davidphilipbarr/36keys Modded by u/gerrycave1"
Changed lines of the file:
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@@
-(kicad_pcb (version 20171130) (host pcbnew "(5.1.9)-1")
+(kicad_pcb (version 20171130) (host pcbnew "(5.1.10)-1")
   (general
     (thickness 1.6)
-    (drawings 36)
+    (drawings 38)
     (tracks 629)
     (zones 0)
@@
   )
   (layers
-    (0 F.Cu signal)
-    (31 B.Cu signal)
-    (32 B.Adhes user)
-    (33 F.Adhes user)
-    (34 B.Paste user)
-    (35 F.Paste user)
+    (0 F.Cu signal hide)
+    (31 B.Cu signal hide)
+    (32 B.Adhes user hide)
+    (33 F.Adhes user hide)
+    (34 B.Paste user hide)
+    (35 F.Paste user hide)
     (36 B.SilkS user)
-    (37 F.SilkS user)
-    (38 B.Mask user)
+    (37 F.SilkS user hide)
+    (38 B.Mask user hide)
     (39 F.Mask user)
-    (40 Dwgs.User user)
-    (41 Cmts.User user)
-    (42 Eco1.User user)
-    (43 Eco2.User user)
+    (40 Dwgs.User user hide)
+    (41 Cmts.User user hide)
+    (42 Eco1.User user hide)
+    (43 Eco2.User user hide)
     (44 Edge.Cuts user)
-    (45 Margin user)
+    (45 Margin user hide)
     (46 B.CrtYd user)
     (47 F.CrtYd user)
-    (48 B.Fab user)
-    (49 F.Fab user)
+    (48 B.Fab user hide)
+    (49 F.Fab user hide)
   )
   (setup
@@
     (pad "" np_thru_hole circle (at -5.5 0) (size 1.7018 1.7018) (drill 1.7018) (layers *.Cu *.Mask))
   )
+  (gr_text "ChocoCorne\ndavidphilipbarr/36keys\nModded by u/gerrycave1" (at 104.14 105.41) (layer B.SilkS)
+    (effects (font (size 1 1) (thickness 0.15)) (justify mirror))
+  )
+  (gr_text "ChocoCorne\ndavidphilipbarr/36keys\nModded by u/gerrycave1" (at 104.14 104.14) (layer F.SilkS)
+    (effects (font (size 1 1) (thickness 0.15) italic))
+  )
   (gr_line (start 77.81952 109.21402) (end 58.71 109.21) (angle 90) (layer Edge.Cuts) (width 0.15))
