File: 42Keys/chocorne/chococorne.kicad_pcb (KiCad board)
At the start: 2 copper layers, 130 x 87.7 mm, 63 parts, among them J1 MJ-4PP-9, J2 OLED, SW1 SW_PUSH, SW10 SW_PUSH, SW11 SW_PUSH, SW12 SW_PUSH, SW13 SW_PUSH, SW14 SW_PUSH, SW15 SW_PUSH, SW16 SW_PUSH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

Commit message: NPTH hole on 6th column tab
Parts:
- removed the h2 at (76.9, 91.3)
- removed the h2 at (76.9, 74.2)
- added REF**: Mounting_Wuerth_WA-SMSI-M1.6_H2.5mm_ThreadDepth1.5mm_NoNPTH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, Mounting_Wuerth:Mounting_Wuerth_WA-SMSI-M1.6_H2.5mm_ThreadDepth1.5mm_NoNPTH_97730256330, F.Cu at (76.9, 91.3)
- added REF**: Mounting_Wuerth_WA-SMSI-M1.6_H2.5mm_ThreadDepth1.5mm_NoNPTH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, Mounting_Wuerth:Mounting_Wuerth_WA-SMSI-M1.6_H2.5mm_ThreadDepth1.5mm_NoNPTH_97730256330, F.Cu at (76.9, 74.1)
